Commit message: fase3 rematada sin main

File: src/p1/barrier.urdf (robot description, URDF)
Before this commit: robot myrobot, 2 links, 1 joints
Links:
- link body_link: mass 5.0 -> 5000.0
- link end_link: mass 1.0 -> 5; geometry collision box size=3 0.1 0.1; visual box size=3 0.1 0.1
Joints:
- joint body_to_end: origin xyz=0.05 0 0.1 -> xyz=0 0 0.1

File: src/p1/rampa.urdf (robot description, URDF)
Before this commit: robot myrobot, 3 links, 2 joints
Links:
- link left: geometry collision box size=4 3.40 0.001; visual box size=4 3.40 0.001
- link right: geometry collision box size=4 3.40 0.001; visual box size=4 3.40 0.001
Joints:
- joint base_to_body: origin xyz=0 0 1.3 rpy=0.785 0 0 -> xyz=0 0 0.8 rpy=0.436332 0 0
- joint base_to_body_2: origin xyz=0 0 1.3 rpy=-0.785 0 0 -> xyz=0 0 0.8 rpy=-0.436332 0 0
